File: BatMeas5.2 JST.sch (EAGLE design)
At the start: 50 parts, among them IC1 ATTINY24, IC2 3V3, IC3 3V, J3 BM03B-PASS-1-TFT_(LF)(SN), J4 BM05B-PASS-1-TFT_(LF)(SN)SMD, T1 MMUN2233, T2 MMUN2233, T3 MMUN2233, T4 MMUN2111LT1G, T5 MMUN2111LT1G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

Commit message: Minor updates and added maunfacturing files
Parts:
- D3: value (none) -> MM3Z3V0ST1G
Other:
- note removed: "D3: 3V Zener for first board MM3Z3V0ST1G"
Changed lines of the file:
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@@
 <part name="LED4" library="led" deviceset="LED" device="CHIPLED_0805" value="150060GS75000"/>
 <part name="D2" library="adafruit" deviceset="DIODE" device="SOD-323F"/>
-<part name="D3" library="adafruit" deviceset="DIODE" device="SOD-323F"/>
+<part name="D3" library="adafruit" deviceset="DIODE" device="SOD-323F" value="MM3Z3V0ST1G "/>
 <part name="J1" library="con-amp" deviceset="MTA05-100" device=""/>
 <part name="GND9" library="supply1" deviceset="GND" device=""/>
@@
 <text x="81.28" y="-41.91" size="1.778" layer="91">R5: Only populate on first board</text>
 <text x="71.12" y="-7.62" size="1.778" layer="91">R6: Populate on all but first board</text>
-<text x="38.1" y="-53.34" size="1.778" layer="91">D3: 3V Zener for first
-board MM3Z3V0ST1G</text>
 <text x="160.02" y="-83.82" size="2.54" layer="91">5.2</text>
 <text x="71.12" y="-67.31" size="3.81" layer="91">(C) 2019 Johannes Huebner
@@
 </instance>
 <instance part="D3" gate="G$1" x="50.8" y="-40.64" smashed="yes" rot="R90">
-<attribute name="NAME" x="48.26" y="-40.64" size="1.27" layer="95" rot="R180"/>
-<attribute name="VALUE" x="54.61" y="-43.18" size="1.27" layer="96" rot="R90"/>
+<attribute name="NAME" x="48.26" y="-38.1" size="1.27" layer="95" rot="R180"/>
+<attribute name="VALUE" x="48.26" y="-40.64" size="1.27" layer="96" rot="R180"/>
 </instance>
 <instance part="J1" gate="G$1" x="-101.6" y="66.04" smashed="yes" rot="R90">
