File: Isolator2.0.sch (EAGLE design)
At the start: 30 parts, among them IC1 MEGA8-AI, IC2 RS485SOIC, J1 RJ45-8PTH, J2 RJ45-8PTH, T3 BC847ALT1SMD

Commit message: Updated Isolator board and added manufacturing files
Other:
- note added: "(C) 2019 Johannes Huebner openinverter.org"
- note added: "2.0"
- note added: "25 July 2019"
- note added: "Isolator PCB"
- moved on the sheet: J1, J2
