File: BatMeas5.3 JST.sch (EAGLE design)
At the start: 50 parts, among them IC1 ATTINY24, IC2 3V3, IC3 3V, J4 BM05B-PASS-1-TFT_(LF)(SN)SMD, T1 MMUN2233, T2 MMUN2233, T3 MMUN2233, T4 MMUN2111LT1G, T5 MMUN2111LT1G, T6 MMUN2111LT1G, T7 MMUN2233, T8 MMUN2233

Commit message: Replaced JST comms connector by AVX or 4mm IDC wire to board connector Removed all THT options Removed holes below cell JST connector, made pads longer
Parts:
- removed J1: (no value), con-amp:MTA05-100
- removed J2: (no value), con-amp:MTA03-100
- removed J3: (no value), adafruit:JST_3PIN
- added X1: 009175003, con-avx:009175003
- added X1_: 4400W03J7923, con-avx:4400W03J7923
Connections:
- net GND: no longer J1.1
- net N$12: now also X1.1@1, X1_.1; no longer J2.1, J3.1
- net N$17: no longer J1.5
- net N$22: now also X1.3@2, X1_.3; no longer J2.3, J3.3
- net N$23: no longer J1.4
- net N$24: no longer J1.3
- net N$25: no longer J1.2
- net TX: now also X1.2@1, X1_.2; no longer J2.2, J3.2
Changed lines of the file:
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@@
 <part name="LED4" library="led" deviceset="LED" device="CHIPLED_0805" value="150060GS75000"/>
 <part name="D2" library="adafruit" deviceset="DIODE" device="SOD-323F" value="1N4148WS"/>
-<part name="J1" library="con-amp" deviceset="MTA05-100" device=""/>
 <part name="GND9" library="supply1" deviceset="GND" device=""/>
 <part name="C6" library="rcl" deviceset="C-EU" device="C0603" value="100n"/>
 <part name="GND12" library="supply1" deviceset="GND" device=""/>
-<part name="J2" library="con-amp" deviceset="MTA03-100" device=""/>
 <part name="R13" library="rcl" deviceset="R-EU_" device="R0603" value="220"/>
 <part name="IC2" library="SparkFun-PowerIC" deviceset="V_REG_LDO" device="SMD" value="3V3"/>
 <part name="IC3" library="SparkFun-PowerIC" deviceset="V_REG_LDO" device="SMD" value="3V"/>
-<part name="J3" library="adafruit" deviceset="JST_3PIN" device=""/>
 <part name="J4" library="BM03B-PASS-1-TFT_(LF)(SN)" deviceset="BM05B-PASS-1-TFT_(LF)(SN)" device="SMD"/>
 <part name="GND14" library="supply1" deviceset="GND" device=""/>
@@
 <part name="D3" library="adafruit" deviceset="DIODE" device="SOD-323F" value="1N4148WS"/>
 <part name="C7" library="rcl" deviceset="C-EU" device="C0805" value="10µ"/>
+<part name="X1" library="con-avx" deviceset="009175003" device=""/>
+<part name="X1_" library="con-avx" deviceset="4400W03J7923" device=""/>
 </parts>
 <sheets>
@@
 <attribute name="VALUE" x="48.26" y="107.95" size="1.27" layer="96"/>
 </instance>
-<instance part="J1" gate="G$1" x="-101.6" y="66.04" smashed="yes" rot="R90">
-<attribute name="NAME" x="-99.06" y="76.2" size="1.778" layer="95" rot="R180"/>
-<attribute name="VALUE" x="-97.79" y="73.66" size="1.778" layer="96" rot="R90"/>
-</instance>
 <instance part="GND9" gate="1" x="2.54" y="73.66" smashed="yes" rot="R180">
 <attribute name="VALUE" x="5.08" y="76.2" size="1.778" layer="96" rot="R180"/>
@@
 <attribute name="VALUE" x="5.08" y="5.08" size="1.778" layer="96"/>
 </instance>
-<instance part="J2" gate="G$1" x="96.52" y="-25.4" smashed="yes" rot="R270">
-<attribute name="NAME" x="96.52" y="-30.48" size="1.778" layer="95" rot="R180"/>
-<attribute name="VALUE" x="92.71" y="-30.48" size="1.778" layer="96" rot="R270"/>
-</instance>
 <instance part="R13" gate="G$1" x="88.9" y="-17.78" smashed="yes" rot="R270">
 <attribute name="NAME" x="82.55" y="-18.8214" size="1.778" layer="95"/>
@@
 <attribute name="NAME" x="12.7" y="65.024" size="1.778" layer="95"/>
 <attribute name="VALUE" x="12.7" y="62.23" size="1.778" layer="96"/>
-</instance>
-<instance part="J3" gate="G$1" x="114.3" y="-25.4" smashed="yes">
-<attribute name="NAME" x="128.27" y="-25.4" size="1.778" layer="95" align="center-left"/>
-<attribute name="VALUE" x="128.27" y="-27.94" size="1.778" layer="96" align="center-left" display="off"/>
 </instance>
 <instance part="J4" gate="G$1" x="-101.6" y="121.92" smashed="yes" rot="R270">
@@
 <attribute name="VALUE" x="92.964" y="-42.799" size="1.778" layer="96"/>
 </instance>
+<instance part="X1" gate="G$1" x="106.68" y="-38.1" rot="R270"/>
+<instance part="X1_" gate="G$1" x="114.3" y="-22.86"/>
 </instances>
 <busses>
@@
 <wire x1="-96.52" y1="15.24" x2="-96.52" y2="60.96" width="0.1524" layer="91"/>
 <wire x1="-96.52" y1="60.96" x2="-99.06" y2="60.96" width="0.1524" layer="91"/>
-<pinref part="J1" gate="G$1" pin="1"/>
 </segment>
 <segment>
@@
 <wire x1="-121.92" y1="68.58" x2="-106.68" y2="68.58" width="0.1524" layer="91"/>
 <pinref part="LED2" gate="G$1" pin="A"/>
-<wire x1="-106.68" y1="68.58" x2="-99.06" y2="68.58" width="0.1524" layer="91"/>
-<wire x1="-99.06" y1="68.58" x2="-88.9" y2="68.58" width="0.1524" layer="91"/>
+<wire x1="-106.68" y1="68.58" x2="-88.9" y2="68.58" width="0.1524" layer="91"/>
 <pinref part="T4" gate="G$1" pin="C"/>
 <wire x1="-121.92" y1="78.74" x2="-127" y2="78.74" width="0.1524" layer="91"/>
@@
 <wire x1="-121.92" y1="83.82" x2="-121.92" y2="78.74" width="0.1524" layer="91"/>
 <junction x="-121.92" y="78.74"/>
-<pinref part="J1" gate="G$1" pin="4"/>
-<junction x="-99.06" y="68.58"/>
 <wire x1="-106.68" y1="68.58" x2="-106.68" y2="104.14" width="0.1524" layer="91"/>
 <wire x1="-106.68" y1="104.14" x2="-99.06" y2="104.14" width="0.1524" layer="91"/>
@@
 <wire x1="-91.44" y1="45.72" x2="-91.44" y2="66.04" width="0.1524" layer="91"/>
 <pinref part="LED3" gate="G$1" pin="A"/>
-<wire x1="-91.44" y1="66.04" x2="-99.06" y2="66.04" width="0.1524" layer="91"/>
 <pinref part="T5" gate="G$1" pin="C"/>
-<wire x1="-99.06" y1="66.04" x2="-109.22" y2="66.04" width="0.1524" layer="91"/>
+<wire x1="-91.44" y1="66.04" x2="-109.22" y2="66.04" width="0.1524" layer="91"/>
 <wire x1="-109.22" y1="66.04" x2="-124.46" y2="66.04" width="0.1524" layer="91"/>
 <wire x1="-124.46" y1="66.04" x2="-124.46" y2="63.5" width="0.1524" layer="91"/>
@@
 <wire x1="-124.46" y1="68.58" x2="-124.46" y2="66.04" width="0.1524" layer="91"/>
 <junction x="-124.46" y="66.04"/>
-<pinref part="J1" gate="G$1" pin="3"/>
-<junction x="-99.06" y="66.04"/>
 <wire x1="-109.22" y1="66.04" x2="-109.22" y2="106.68" width="0.1524" layer="91"/>
 <junction x="-109.22" y="66.04"/>
@@
 <pinref part="LED4" gate="G$1" pin="A"/>
 <wire x1="-114.3" y1="63.5" x2="-111.76" y2="63.5" width="0.1524" layer="91"/>
-<wire x1="-111.76" y1="63.5" x2="-99.06" y2="63.5" width="0.1524" layer="91"/>
-<wire x1="-99.06" y1="63.5" x2="-93.98" y2="63.5" width="0.1524" layer="91"/>
+<wire x1="-111.76" y1="63.5" x2="-93.98" y2="63.5" width="0.1524" layer="91"/>
 <wire x1="-114.3" y1="48.26" x2="-127" y2="48.26" width="0.1524" layer="91"/>
 <pinref part="T6" gate="G$1" pin="C"/>
 <wire x1="-157.48" y1="53.34" x2="-114.3" y2="53.34" width="0.1524" layer="91"/>
 <junction x="-114.3" y="53.34"/>
-<pinref part="J1" gate="G$1" pin="2"/>
-<junction x="-99.06" y="63.5"/>
 <wire x1="-111.76" y1="63.5" x2="-111.76" y2="109.22" width="0.1524" layer="91"/>
 <junction x="-111.76" y="63.5"/>
@@
 <wire x1="-119.38" y1="71.12" x2="-104.14" y2="71.12" width="0.1524" layer="91"/>
 <pinref part="LED1" gate="G$1" pin="A"/>
-<wire x1="-104.14" y1="71.12" x2="-99.06" y2="71.12" width="0.1524" layer="91"/>
-<wire x1="-99.06" y1="71.12" x2="-88.9" y2="71.12" width="0.1524" layer="91"/>
+<wire x1="-104.14" y1="71.12" x2="-88.9" y2="71.12" width="0.1524" layer="91"/>
 <wire x1="-119.38" y1="93.98" x2="-127" y2="93.98" width="0.1524" layer="91"/>
 <wire x1="-88.9" y1="111.76" x2="-88.9" y2="86.36" width="0.1524" layer="91"/>
 <junction x="-88.9" y="86.36"/>
-<pinref part="J1" gate="G$1" pin="5"/>
-<junction x="-99.06" y="71.12"/>
 <wire x1="-104.14" y1="71.12" x2="-104.14" y2="101.6" width="0.1524" layer="91"/>
 <junction x="-104.14" y="71.12"/>
@@
 <wire x1="7.62" y1="-20.32" x2="83.82" y2="-20.32" width="0.1524" layer="91"/>
 <wire x1="83.82" y1="-20.32" x2="83.82" y2="-25.4" width="0.1524" layer="91"/>
-<pinref part="J2" gate="G$1" pin="2"/>
-<wire x1="93.98" y1="-25.4" x2="83.82" y2="-25.4" width="0.1524" layer="91"/>
-<pinref part="J3" gate="G$1" pin="2"/>
-<wire x1="93.98" y1="-25.4" x2="111.76" y2="-25.4" width="0.1524" layer="91"/>
-<junction x="93.98" y="-25.4"/>
+<pinref part="X1_" gate="G$1" pin="2"/>
+<wire x1="83.82" y1="-25.4" x2="104.14" y2="-25.4" width="0.1524" layer="91"/>
+<pinref part="X1" gate="G$1" pin="2@1"/>
+<wire x1="104.14" y1="-25.4" x2="111.76" y2="-25.4" width="0.1524" layer="91"/>
+<wire x1="104.14" y1="-33.02" x2="104.14" y2="-25.4" width="0.1524" layer="91"/>
+<junction x="104.14" y="-25.4"/>
 </segment>
 </net>
@@
 <segment>
 <pinref part="R13" gate="G$1" pin="2"/>
-<pinref part="J2" gate="G$1" pin="1"/>
-<wire x1="88.9" y1="-22.86" x2="93.98" y2="-22.86" width="0.1524" layer="91"/>
-<pinref part="J3" gate="G$1" pin="1"/>
-<wire x1="93.98" y1="-22.86" x2="111.76" y2="-22.86" width="0.1524" layer="91"/>
-<junction x="93.98" y="-22.86"/>
 <pinref part="C7" gate="G$1" pin="1"/>
 <wire x1="88.9" y1="-35.56" x2="88.9" y2="-22.86" width="0.1524" layer="91"/>
 <junction x="88.9" y="-22.86"/>
+<pinref part="X1_" gate="G$1" pin="1"/>
+<wire x1="88.9" y1="-22.86" x2="106.68" y2="-22.86" width="0.1524" layer="91"/>
+<pinref part="X1" gate="G$1" pin="1@1"/>
+<wire x1="106.68" y1="-22.86" x2="111.76" y2="-22.86" width="0.1524" layer="91"/>
+<wire x1="106.68" y1="-33.02" x2="106.68" y2="-22.86" width="0.1524" layer="91"/>
+<junction x="106.68" y="-22.86"/>
 </segment>
 </net>
 <net name="N$22" class="0">
 <segment>
-<pinref part="J2" gate="G$1" pin="3"/>
-<wire x1="93.98" y1="-27.94" x2="78.74" y2="-27.94" width="0.1524" layer="91"/>
 <pinref part="R12" gate="G$1" pin="2"/>
-<pinref part="J3" gate="G$1" pin="3"/>
-<wire x1="93.98" y1="-27.94" x2="111.76" y2="-27.94" width="0.1524" layer="91"/>
-<junction x="93.98" y="-27.94"/>
-</segment>
-</net>
+<pinref part="X1_" gate="G$1" pin="3"/>
+<wire x1="78.74" y1="-27.94" x2="101.6" y2="-27.94" width="0.1524" layer="91"/>
+<pinref part="X1" gate="G$1" pin="3@2"/>
+<wire x1="101.6" y1="-27.94" x2="111.76" y2="-27.94" width="0.1524" layer="91"/>
+<wire x1="101.6" y1="-33.02" x2="101.6" y2="-27.94" width="0.1524" layer="91"/>
+<junction x="101.6" y="-27.94"/>
+</segment>
+</net>

Commit message: Updated BOM
Parts:
- C5: value 4n7 -> 10n
Changed lines of the file:
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@@
 <part name="R6" library="rcl" deviceset="R-EU_" device="R0603" value="1k"/>
 <part name="R11" library="rcl" deviceset="R-EU_" device="R0603" value="220"/>
-<part name="C5" library="rcl" deviceset="C-EU" device="C0603" value="4n7"/>
+<part name="C5" library="rcl" deviceset="C-EU" device="C0603" value="10n"/>
 <part name="GND16" library="supply1" deviceset="GND" device=""/>
 <part name="R12" library="rcl" deviceset="R-EU_" device="R0603" value="220"/>
@@
 </segment>
 <segment>
-<wire x1="-96.52" y1="15.24" x2="-68.58" y2="15.24" width="0.1524" layer="91"/>
-<junction x="-68.58" y="15.24"/>
 <pinref part="C1" gate="G$1" pin="2"/>
 <pinref part="GND2" gate="1" pin="GND"/>
-<wire x1="-96.52" y1="15.24" x2="-96.52" y2="60.96" width="0.1524" layer="91"/>
-<wire x1="-96.52" y1="60.96" x2="-99.06" y2="60.96" width="0.1524" layer="91"/>
 </segment>
 <segment>
